File: OffsetAttenuator.kicad_pcb (KiCad board)
At the start: 2 copper layers, 0 parts

Commit message: schematic updates
Parts:
- added BT1: Battery 9V, Library:1294PCB_29P57X53P85_KEY, F.Cu at (112.9, 69.9)
- added C1: 470pF, Capacitor_THT:C_Disc_D5.0mm_W2.5mm_P5.00mm, F.Cu at (145.7, 104.7)
- added C2: 470pF, Capacitor_THT:C_Disc_D5.0mm_W2.5mm_P5.00mm, F.Cu at (145.7, 108.8)
- added C3: .0047uF, Capacitor_THT:C_Disc_D5.0mm_W2.5mm_P5.00mm, F.Cu at (145.7, 112.8)
- added D1: 1N4148, Diode_THT:D_DO-35_SOD27_P7.62mm_Horizontal, F.Cu at (153.9, 121.5)
- added D2: LED, LED_THT:LED_D5.0mm, F.Cu at (146.6, 118.6)
- added J1: Conn_Coaxial, Library:CONBNC002, F.Cu at (137.8, 77.1)
- added J2: Conn_Coaxial, Library:CONBNC002, F.Cu at (153.8, 77.1)
- added R1: 2.2K, Resistor_THT:R_Axial_DIN0309_L9.0mm_D3.2mm_P12.70mm_Horizontal, F.Cu at (136.4, 86.1)
- added R3: 2.2K, Resistor_THT:R_Axial_DIN0309_L9.0mm_D3.2mm_P12.70mm_Horizontal, F.Cu at (136.4, 90.8)
- added R4: 4.7K, Resistor_THT:R_Axial_DIN0309_L9.0mm_D3.2mm_P12.70mm_Horizontal, F.Cu at (136.4, 95.6)
- added R5: 220, Resistor_THT:R_Axial_DIN0309_L9.0mm_D3.2mm_P12.70mm_Horizontal, F.Cu at (136.4, 100.3)
- added RV1: 5K, Library:TRIM_3310Y-001-502L, F.Cu at (158.4, 108.2)
- added SW1: POWER, Library:SWT3, F.Cu at (137.3, 105.9)
- added SW2: BYPASS, Library:SWT3, F.Cu at (137.3, 112.2)
- added U1: L7805, Package_TO_SOT_THT:TO-220-3_Vertical, F.Cu at (155.5, 117.7)
- added X1: 4MHz, Library:OSC_ECS-2100AX-040, F.Cu at (158.6, 91.1)
