File: OffsetAttenuator.kicad_pcb (KiCad board)
At the start: 2 copper layers, 92.5 x 65 mm, 21 parts, among them J1 Conn_Coaxial, J2 Conn_Coaxial, SW1 POWER, SW2 BYPASS, U1 L7805, Y1 ECS-2100AX-040

Commit message: updating silkscreen
Other:
- board text added: "FoxHunt Offset Attenuator"
- board text added: "https://www.w9dup.org/test_eqpt_files/attenuator_project_2010_may.pdf"
Changed lines of the file:
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@@
 		(layer "Edge.Cuts")
+	)
+	(gr_text "https://www.w9dup.org/test_eqpt_files/attenuator_project_2010_may.pdf"
+		(at 36.6 78.3 0)
+		(layer "F.SilkS")
+		(effects
+			(font
+				(size 1.5 1.5)
+				(thickness 0.3)
+				(bold yes)
+			)
+			(justify left bottom)
+		)
+	)
+	(gr_text "FoxHunt Offset Attenuator"
+		(at 64.2 24 0)
+		(layer "F.SilkS")
+		(effects
+			(font
+				(size 1.5 1.5)
+				(thickness 0.3)
+				(bold yes)
+			)
+			(justify left bottom)
+		)
 	)
 	(segment

Commit message: adding gerbers
Other:
- board text added: "BYPASS"
- board text added: "POWER"
Changed lines of the file:
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@@
 			(plot_on_all_layers_selection 0x00000000_00000000_00000000_00000000)
 			(disableapertmacros no)
-			(usegerberextensions no)
+			(usegerberextensions yes)
 			(usegerberattributes yes)
 			(usegerberadvancedattributes yes)
@@
 			(sketchdnponfab yes)
 			(crossoutdnponfab yes)
-			(subtractmaskfromsilk no)
+			(subtractmaskfromsilk yes)
 			(outputformat 1)
 			(mirror no)
-			(drillshape 1)
+			(drillshape 0)
 			(scaleselection 1)
-			(outputdirectory "")
+			(outputdirectory "Gerbers/")
 		)
 	)
@@
 			)
 			(justify left bottom)
+		)
+	)
+	(gr_text "POWER"
+		(at 49.5 58.5 90)
+		(layer "F.SilkS")
+		(effects
+			(font
+				(size 1 1)
+				(thickness 0.1)
+			)
+			(justify left bottom)
+		)
+	)
+	(gr_text "BYPASS"
+		(at 49.5 49.5 90)
+		(layer "F.SilkS")
+		(effects
+			(font
+				(size 1 1)
+				(thickness 0.1)
+			)
+			(justify left bottom)
